File: hardware/bareboard/bareboard.kicad_pcb (KiCad board)
At the start: 6 copper layers, 95.9 x 90.2 mm, 5 parts, among them J1 Conn_02x20_Odd_Even

Commit message: bareboard: update holes to be H1-H4
Instead of H101-H104 as they were before.
Parts:
- renumbered H101 to H1, H102 to H2, H103 to H3, H104 to H4
Changed lines of the file:
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@@
 		(descr "Mounting Hole 3.2mm, M3, DIN965")
 		(tags "mounting hole 3.2mm m3 din965")
-		(property "Reference" "H102"
+		(property "Reference" "H2"
 			(at 0 -3.8 180)
 			(layer "F.SilkS")
@@
 		(descr "Mounting Hole 3.2mm, M3, DIN965")
 		(tags "mounting hole 3.2mm m3 din965")
-		(property "Reference" "H101"
+		(property "Reference" "H1"
 			(at 0 -3.8 180)
 			(layer "F.SilkS")
@@
 		(descr "Mounting Hole 3.2mm, M3, DIN965")
 		(tags "mounting hole 3.2mm m3 din965")
-		(property "Reference" "H104"
+		(property "Reference" "H4"
 			(at 0 -3.8 180)
 			(layer "F.SilkS")
@@
 		(descr "Mounting Hole 3.2mm, M3, DIN965")
 		(tags "mounting hole 3.2mm m3 din965")
-		(property "Reference" "H103"
+		(property "Reference" "H3"
 			(at 0 -3.8 180)
 			(layer "F.SilkS")
