File: hardware/cpb/PairPowerSwitches.kicad_sch (KiCad schematic)
At the start: 5 parts, among them Q24 MBT2222ADW1T1, Q25 IRF7306

Commit message: cpb: Bill of materials updates
One layout change will result: some 1206 resistors became 2012.
Parts:
- R96, R97: LCSC (none) -> C844918
- RN4: LCSC (none) -> C327044
Changed lines of the file:
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@@
+			)
+		)
+		(property "LCSC" "C327044"
+			(at 120.65 64.77 0)
+			(effects
+				(font
+					(size 1.27 1.27)
+				)
+				(hide yes)
 			)
 		)
@@
 		)
 		(property "Description" "4 resistor network, parallel topology, split"
+			(at 50.8 59.69 0)
+			(effects
+				(font
+					(size 1.27 1.27)
+				)
+				(hide yes)
+			)
+		)
+		(property "LCSC" "C327044"
 			(at 50.8 59.69 0)
 			(effects
@@
 			)
 		)
+		(property "LCSC" "C844918"
+			(at 124.46 45.72 0)
+			(effects
+				(font
+					(size 1.27 1.27)
+				)
+				(hide yes)
+			)
+		)
 		(pin "2"
 		)
@@
 			)
 		)
+		(property "LCSC" "C844918"
+			(at 59.69 45.72 0)
+			(effects
+				(font
+					(size 1.27 1.27)
+				)
+				(hide yes)
+			)
+		)
 		(pin "2"
 		)
@@
 			)
 		)
+		(property "LCSC" "C327044"
+			(at 55.88 64.77 0)
+			(effects
+				(font
+					(size 1.27 1.27)
+				)
+				(hide yes)
+			)
+		)
 		(pin "4"
 		)
@@
 			(at 115.57 59.69 0)
 			(effects
+				(font
+					(size 1.27 1.27)
+				)
+				(hide yes)
+			)
+		)
+		(property "LCSC" "C327044"
+			(at 115.57 59.69 0)
+			(effects
