File: hardware/cpb/FourFullBridges.kicad_sch (KiCad schematic)
At the start: 31 parts, among them Q5 PMBT2222A, Q6 IRF9393, Q7 PMBT2222A, U7 SC18IS606, U8 KF33BDT, U9 MAX22200

Commit message: cpb: update part numbers and attributes
Parts:
- D10, D11, D8, D9: LCSC C22582 -> C604793
Changed lines of the file:
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@@
 			)
 		)
-		(property "LCSC" "C22582"
+		(property "LCSC" "C604793"
 			(at 22.86 187.96 0)
 			(effects
@@
 			)
 		)
-		(property "LCSC" "C22582"
+		(property "LCSC" "C604793"
 			(at 95.25 187.96 0)
 			(effects
@@
 			)
 		)
-		(property "LCSC" "C22582"
+		(property "LCSC" "C604793"
 			(at 130.81 187.96 0)
 			(effects
@@
 			)
 		)
-		(property "LCSC" "C22582"
+		(property "LCSC" "C604793"
 			(at 58.42 187.96 0)
 			(effects
